Commit message: Clean up grasp planner

File: src/pb_robot/models/franka_description/robots/hand.urdf (robot description, URDF)
Before this commit: robot hand, 4 links, 3 joints
Links:
- link panda_leftfinger: geometry collision mesh filename=package://franka_description/meshes/collision/finger.stl; visual mesh filename=package://franka_description/meshes/collision/finger.stl
- link panda_rightfinger: geometry collision mesh filename=package://franka_description/meshes/collision/finger.stl; visual mesh filename=package://franka_description/meshes/collision/finger.stl

Commit message: Update finger geom

File: src/pb_robot/models/franka_description/robots/hand.urdf (robot description, URDF)
Before this commit: robot hand, 4 links, 3 joints
Links:
- link panda_leftfinger: geometry collision mesh filename=package://franka_description/meshes/visual/finger.dae; visual mesh filename=package://franka_description/meshes/visual/finger.dae
- link panda_rightfinger: geometry collision mesh filename=package://franka_description/meshes/visual/finger.dae; visual mesh filename=package://franka_description/meshes/visual/finger.dae
