Commit message: Add wrist camera model

File: src/pb_robot/models/franka_description/robots/panda_arm_hand.urdf (robot description, URDF)
Before this commit: robot panda, 13 links, 12 joints
Links:
- added link camera_bottom_screw_frame
- added link camera_color_frame
- added link camera_color_optical_frame
- added link camera_link, mass 0.072; collision box size=0.02505 0.09 0.025; visual box size=0.09 0.025 0.02505
Joints:
- added joint camera_color_joint: type fixed, parent camera_link, child camera_color_frame, origin xyz=0 0.015 0 rpy=0 0 0
- added joint camera_color_optical_joint: type fixed, parent camera_color_frame, child camera_color_optical_frame, origin xyz=0 0 0 rpy=-1.57079632679 0 -1.57079632679
- added joint camera_joint: type fixed, parent panda_hand, child camera_bottom_screw_frame, origin xyz= 0.09217904 -0.00621438 -0.0266488 rpy=-0.00708276 -1.03952579  3.11958769
- added joint camera_link_joint: type fixed, parent camera_bottom_screw_frame, child camera_link, origin xyz=0.0106 0.0175 0.0125 rpy=0 0 0

Commit message: Update camera location in sim

File: src/pb_robot/models/franka_description/robots/panda_arm_hand.urdf (robot description, URDF)
Before this commit: robot panda, 17 links, 16 joints
Joints:
- joint camera_joint: origin xyz= 0.09217904 -0.00621438 -0.0266488 rpy=-0.00708276 -1.03952579  3.11958769 -> xyz=0.02680958 0.00117613 0.04814077 rpy=-0.06882249 -1.40188346 -3.07369552

Commit message: Fix bug in calculating location of hand for grasp. Should be centered 1cm in from each edge now

File: src/pb_robot/models/franka_description/robots/panda_arm_hand.urdf (robot description, URDF)
Before this commit: robot panda, 17 links, 16 joints
Joints:
- joint camera_joint: origin xyz=0.02680958 0.00117613 0.04814077 rpy=-0.06882249 -1.40188346 -3.07369552 -> xyz=0.02680958 0.00117613 0.02814077 rpy=-0.06882249 -1.40188346 -3.07369552

Commit message: Add larger fingers to URDF for collision avoidance

File: src/pb_robot/models/franka_description/robots/panda_arm_hand.urdf (robot description, URDF)
Before this commit: robot panda, 17 links, 16 joints
Links:
- link panda_leftfinger: geometry collision box size=0.025 0.025 0.05; visual box size=0.025 0.025 0.05
- link panda_rightfinger: geometry collision box size=0.025 0.025 0.05; visual box size=0.025 0.025 0.05

Commit message: modify placement

File: src/pb_robot/models/franka_description/robots/panda_arm_hand.urdf (robot description, URDF)
Before this commit: robot panda, 17 links, 16 joints
Links:
- link panda_leftfinger: geometry collision box size=0.025 0.025 0.025; visual box size=0.025 0.025 0.025
- link panda_rightfinger: geometry collision box size=0.025 0.025 0.025; visual box size=0.025 0.025 0.025
